File: PCBs/Back/Back.kicad_pcb (KiCad board)
At the start: 2 copper layers, 82 x 82 mm, 146 parts, among them J1 PWR_CONN, J3 TC2030, J4 CAP_CONN, U1 CH32V003F4U6

Commit message: Almost final adjustments
Parts:
- added G***: LOGO, LOGO, B.Cu at (110.0, 94.4)
- added H1: Tooling, fp:ToolingHole, F.Cu at (110.0, 120.6)
- added H2: Tooling, fp:ToolingHole, F.Cu at (71.7, 60.5)
- added H3: Tooling, fp:ToolingHole, F.Cu at (148.3, 60.4)
- R2: value 22k -> 10k
- moved R5 7.03 mm to (80.1, 71.1)
- moved R6 6.75 mm to (80.1, 73.9)
- moved R7 6.75 mm to (80.1, 76.7)
- moved BZ1 3.35 mm to (122.1, 56.5)
- moved J3 1.13 mm to (96.7, 44.0)
- moved R1 0.80 mm to (110.0, 43.0)
- moved C65 0.61 mm to (113.1, 52.0)
- moved C66 0.61 mm to (114.6, 52.0)
- moved R2 0.60 mm to (110.0, 46.1)
Routing:
- net +5V: track 99.1 -> 110.4 mm, vias 0 -> 4
- net /TOUCH3: track 58.5 -> 64.0 mm, vias 4 -> 2
- net /TOUCH2: track 57.7 -> 62.9 mm
- net /TOUCH1: track 57.1 -> 61.9 mm
- net /BUZ: track 25.0 -> 23.1 mm
- net GND: track 133.9 -> 135.7 mm
- net /TX: track 17.9 -> 16.8 mm
- net /SWIO: track 14.7 -> 13.5 mm
- net /RX: track 16.3 -> 15.1 mm
- net /DIN: track 33.0 -> 34.1 mm
- net /LDR_DIV: track 5.91 -> 6.89 mm
Other:
- board text added: "1"
- board text added: "A. Anderson D. Quach J. Wheeler"
- board text added: "Christmas Card 2023 CH32 Fireplace"
- board text added: "God jul & Gott nytt år!"

Commit message: Added small instruction text
Other:
- board text added: "JLCJLCJLCJLC"
- board text added: "Press stockings to interact! Scan QR-code for more instructions."
- board text added: "locked"
- board text removed: "Christmas Card 2023 CH32 Fireplace"
