File: PCBs/Back/Back.kicad_sch (KiCad schematic)
At the start: 146 parts, among them J1 PWR_CONN, J3 TC2030, J4 CAP_CONN, U1 CH32V003F4U6

Commit message: Almost final adjustments
Parts:
- added H1, H2, H3: Tooling, fp:ToolingHole, symbol Mechanical:MountingHole
- BZ1: MPN (none) -> C391038
- C1, C10, C11, C12, C13, C14, C15, C16, C17, C18, C19, C2, C20, C21, C22, C23, C24, C25, C26, C27, C28, C29, C3, C30, C31, C32, C33, C34, C35, C36, C37, C38, C39, C4, C40, C41, C42, C43, C44, C45, C46, C47, C48, C49, C5, C50, C51, C52, C53, C54, C55, C56, C57, C58, C59, C6, C60, C61, C62, C63, C64, C65, C66, C7, C8, C9: MPN (none) -> C1525
- D1, D10, D11, D12, D13, D14, D15, D16, D17, D18, D19, D2, D20, D21, D22, D23, D24, D25, D26, D27, D28, D29, D3, D30, D31, D32, D33, D34, D35, D36, D37, D38, D39, D4, D40, D41, D42, D43, D44, D45, D46, D47, D48, D49, D5, D50, D51, D52, D53, D54, D55, D56, D57, D58, D59, D6, D60, D61, D62, D63, D64, D7, D8, D9: MPN (none) -> C5349954
- F1: MPN (none) -> C269105
- R1: MPN (none) -> C2904881
- R2: value 22k -> 10k; LCSC C31850 -> C25804; MPN (none) -> C25804
- R3, R4: MPN (none) -> C23186
- R5, R6, R7: MPN (none) -> C23203
- U1: MPN (none) -> C5299908
Other:
- note added: "Connected to Timer2 CH3"
- note added: "LDR_DIV = R2/(R1+R2)*5V"
- note removed: "Check if 22k works"
- note removed: "Connected to Timer1 CH1"
- note removed: "LDR_DIV = R4/(R3+R4)*5V"

Commit message: Cleaned up schematic and generated pdfs
Other:
- title: (none) -> CH32 Fireplace Back PCB
Changed lines of the file:
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@@
 (kicad_sch (version 20230121) (generator eeschema)
   (paper "A3")
+  (title_block
+    (title "CH32 Fireplace Back PCB")
+  )
   (junction (at 287.02 30.48) (diameter 0) (color 0 0 0 0)
   )
