File: PCBs/Middle/Middle.kicad_sch (KiCad schematic)
At the start: 1 part, among them J1 USB_C_Receptacle_PowerOnly_6P

Commit message: back layout done
Parts:
- added J2, J3: Conn_01x04, symbol Connector_Generic:Conn_01x04
Changed lines of the file:
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@@
+    )
+  )
+  (symbol (lib_id "Connector_Generic:Conn_01x04") (at 101.6 57.15 0) (unit 1)
+    (in_bom yes) (on_board yes) (dnp no) (fields_autoplaced)
+    (property "Reference" "J2" (at 104.14 57.15 0)
+      (effects (font (size 1.27 1.27)) (justify left))
+    )
+    (property "Value" "Conn_01x04" (at 104.14 59.69 0)
+      (effects (font (size 1.27 1.27)) (justify left))
+    )
+    (property "Footprint" "" (at 101.6 57.15 0)
+      (effects (font (size 1.27 1.27)) hide)
+    )
+    (property "Datasheet" "~" (at 101.6 57.15 0)
+      (effects (font (size 1.27 1.27)) hide)
+    )
+    (pin "1")
+    (pin "2")
+    (pin "3")
+    (pin "4")
+    (instances
+      (project "Middle"
+        (path "/5f68482a-35f9-4a1e-8449-fd362c622437"
+          (reference "J2") (unit 1)
+        )
+      )
     )
   )
@@
         )
       )
+    )
+  )
+  (symbol (lib_id "Connector_Generic:Conn_01x04") (at 86.36 77.47 0) (unit 1)
+    (in_bom yes) (on_board yes) (dnp no) (fields_autoplaced)
+    (property "Reference" "J3" (at 88.9 77.47 0)
+      (effects (font (size 1.27 1.27)) (justify left))
+    )
+    (property "Value" "Conn_01x04" (at 88.9 80.01 0)
+      (effects (font (size 1.27 1.27)) (justify left))
+    )
+    (property "Footprint" "" (at 86.36 77.47 0)
+      (effects (font (size 1.27 1.27)) hide)
+    )
+    (property "Datasheet" "~" (at 86.36 77.47 0)
+      (effects (font (size 1.27 1.27)) hide)
+    )
+    (pin "1")
+    (pin "2")
+    (pin "3")
+    (pin "4")
+    (instances
+      (project "Middle"
+        (path "/5f68482a-35f9-4a1e-8449-fd362c622437"
+          (reference "J3") (unit 1)
+        )
+      )

Commit message: Middle pcb done
Parts:
- added TP1: TOUCH1, Library:CapPad, symbol Connector:TestPoint
- added TP2: TOUCH2, Library:CapPad, symbol Connector:TestPoint
- added TP3: TOUCH3, Library:CapPad, symbol Connector:TestPoint
- J2: value Conn_01x04 -> PWR; footprint (none) -> Connector_PinHeader_2.54mm:PinHeader_1x04_P2.54mm_Vertical
- J3: value Conn_01x04 -> CAP_TOUCH; footprint (none) -> Connector_PinHeader_2.54mm:PinHeader_1x04_P2.54mm_Vertical
Connections:
- net +5V: now also J3.1 (Pin_1)
- net CC1: now also J3.3 (Pin_3)
- net CC2: now also J3.4 (Pin_4)
- net GND: now also J2.4 (Pin_4), J3.2 (Pin_2)
- net TOUCH1: now reaches J2.1 (Pin_1)
- net TOUCH1: now also TP1.1
- net TOUCH2: now reaches J2.2 (Pin_2)
- net TOUCH2: now also TP2.1
- net TOUCH3: now reaches J2.3 (Pin_3)
- net TOUCH3: now also TP3.1
Other:
- moved on the sheet: J2, J3

Commit message: fixed step files
Parts:
- TP1, TP2, TP3: footprint Library:CapPad -> cap_sock:cap_sock
Changed lines of the file:
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@@
       (effects (font (size 1.27 1.27)) (justify left))
     )
-    (property "Footprint" "Library:CapPad" (at 207.01 41.91 0)
+    (property "Footprint" "cap_sock:cap_sock" (at 207.01 41.91 0)
       (effects (font (size 1.27 1.27)) hide)
     )
@@
       (effects (font (size 1.27 1.27)) (justify left))
     )
-    (property "Footprint" "Library:CapPad" (at 184.15 41.91 0)
+    (property "Footprint" "cap_sock:cap_sock" (at 184.15 41.91 0)
       (effects (font (size 1.27 1.27)) hide)
     )
@@
       (effects (font (size 1.27 1.27)) (justify left))
     )
-    (property "Footprint" "Library:CapPad" (at 229.87 41.91 0)
+    (property "Footprint" "cap_sock:cap_sock" (at 229.87 41.91 0)
       (effects (font (size 1.27 1.27)) hide)
     )

Commit message: Almost final adjustments
Parts:
- J2: value PWR -> CAPTOUCH
- J3: value CAP_TOUCH -> PWR
Changed lines of the file:
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@@
       (effects (font (size 1.27 1.27)) (justify left))
     )
-    (property "Value" "PWR" (at 144.78 48.26 0)
+    (property "Value" "CAPTOUCH" (at 144.78 48.26 0)
       (effects (font (size 1.27 1.27)) (justify left))
     )
@@
       (effects (font (size 1.27 1.27)) (justify left))
     )
-    (property "Value" "CAP_TOUCH" (at 113.03 48.26 0)
+    (property "Value" "PWR" (at 113.03 48.26 0)
       (effects (font (size 1.27 1.27)) (justify left))
     )

Commit message: Cleaned up schematic and generated pdfs
Other:
- note added: "Board to Board connectors"
- note added: "CC Pins pulled down to 5.1k for standard 5V power negotiation"
- note added: "Capacitive Touch Pads"
- note added: "USB POWER"
- note removed: "Pins"
- note removed: "Usb power"
- moved on the sheet: TP1, TP2, TP3
Changed lines of the file:
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@@
 (kicad_sch (version 20230121) (generator eeschema)
-  (paper "A4")
+  (paper "A5")
   (junction (at 38.1 69.85) (diameter 0) (color 0 0 0 0)
   )
@@
     (stroke (width 0) (type default))
   )
-  (wire (pts (xy 201.93 41.91) (xy 201.93 44.45))
+  (wire (pts (xy 50.8 110.49) (xy 50.8 113.03))
     (stroke (width 0) (type default))
   )
@@
     (stroke (width 0) (type default))
   )
-  (wire (pts (xy 224.79 41.91) (xy 224.79 44.45))
+  (wire (pts (xy 73.66 110.49) (xy 73.66 113.03))
     (stroke (width 0) (type default))
   )
@@
     (stroke (width 0) (type default))
   )
-  (wire (pts (xy 179.07 44.45) (xy 173.99 44.45))
+  (wire (pts (xy 27.94 113.03) (xy 22.86 113.03))
     (stroke (width 0) (type default))
   )
@@
     (stroke (width 0) (type default))
   )
-  (wire (pts (xy 201.93 44.45) (xy 195.58 44.45))
+  (wire (pts (xy 50.8 113.03) (xy 44.45 113.03))
     (stroke (width 0) (type default))
   )
@@
     (stroke (width 0) (type default))
   )
-  (wire (pts (xy 179.07 41.91) (xy 179.07 44.45))
+  (wire (pts (xy 27.94 110.49) (xy 27.94 113.03))
     (stroke (width 0) (type default))
   )
@@
     (stroke (width 0) (type default))
   )
-  (wire (pts (xy 224.79 44.45) (xy 220.98 44.45))
-    (stroke (width 0) (type default))
-  )
-  (text "Usb power" (at 21.59 22.86 0)
+  (wire (pts (xy 73.66 113.03) (xy 69.85 113.03))
+    (stroke (width 0) (type default))
+  )
+  (rectangle (start 12.7 85.09) (end 88.9 134.62)
+    (stroke (width 0) (type default))
+    (fill (type none))
+  )
+  (rectangle (start 80.01 12.7) (end 163.83 85.09)
+    (stroke (width 0) (type default))
+    (fill (type none))
+  )
+  (rectangle (start 12.7 12.7) (end 80.01 85.09)
+    (stroke (width 0) (type default))
+    (fill (type none))
+  )
+  (text "USB POWER" (at 15.24 83.82 0)
     (effects (font (size 2 2)) (justify left bottom))
   )
-  (text "Pins" (at 118.11 29.21 0)
+  (text "Capacitive Touch Pads" (at 13.97 133.35 0)
     (effects (font (size 2 2)) (justify left bottom))
   )
-  (label "TOUCH2" (at 195.58 44.45 180) (fields_autoplaced)
+  (text "CC Pins pulled down to 5.1k for \nstandard 5V power negotiation"
+    (at 46.99 83.82 0)
+    (effects (font (size 1.27 1.27)) (justify left bottom))
+  )
+  (text "Board to Board connectors" (at 81.28 83.82 0)
+    (effects (font (size 2 2)) (justify left bottom))
+  )
+  (label "TOUCH2" (at 44.45 113.03 180) (fields_autoplaced)
     (effects (font (size 1.27 1.27)) (justify right bottom))
   )
@@
     (effects (font (size 1.27 1.27)) (justify left bottom))
   )
-  (label "TOUCH1" (at 173.99 44.45 180) (fields_autoplaced)
+  (label "TOUCH1" (at 22.86 113.03 180) (fields_autoplaced)
     (effects (font (size 1.27 1.27)) (justify right bottom))
   )
@@
     (effects (font (size 1.27 1.27)) (justify right bottom))
   )
-  (label "TOUCH3" (at 220.98 44.45 180) (fields_autoplaced)
+  (label "TOUCH3" (at 69.85 113.03 180) (fields_autoplaced)
     (effects (font (size 1.27 1.27)) (justify right bottom))
   )
@@
     )
   )
-  (symbol (lib_id "Connector:TestPoint") (at 201.93 41.91 0) (unit 1)
-    (in_bom yes) (on_board yes) (dnp no) (fields_autoplaced)
-    (property "Reference" "TP2" (at 204.47 37.338 0)
-      (effects (font (size 1.27 1.27)) (justify left))
-    )
-    (property "Value" "TOUCH2" (at 204.47 39.878 0)
-      (effects (font (size 1.27 1.27)) (justify left))
-    )
-    (property "Footprint" "cap_sock:cap_sock" (at 207.01 41.91 0)
-      (effects (font (size 1.27 1.27)) hide)
-    )
-    (property "Datasheet" "~" (at 207.01 41.91 0)
+  (symbol (lib_id "Connector:TestPoint") (at 50.8 110.49 0) (unit 1)
+    (in_bom yes) (on_board yes) (dnp no) (fields_autoplaced)
+    (property "Reference" "TP2" (at 53.34 105.918 0)
+      (effects (font (size 1.27 1.27)) (justify left))
+    )
+    (property "Value" "TOUCH2" (at 53.34 108.458 0)
+      (effects (font (size 1.27 1.27)) (justify left))
+    )
+    (property "Footprint" "cap_sock:cap_sock" (at 55.88 110.49 0)
+      (effects (font (size 1.27 1.27)) hide)
+    )
+    (property "Datasheet" "~" (at 55.88 110.49 0)
       (effects (font (size 1.27 1.27)) hide)
     )
@@
     )
   )
-  (symbol (lib_id "Connector:TestPoint") (at 179.07 41.91 0) (unit 1)
-    (in_bom yes) (on_board yes) (dnp no) (fields_autoplaced)
-    (property "Reference" "TP1" (at 181.61 37.338 0)
-      (effects (font (size 1.27 1.27)) (justify left))
-    )
-    (property "Value" "TOUCH1" (at 181.61 39.878 0)
-      (effects (font (size 1.27 1.27)) (justify left))
-    )
-    (property "Footprint" "cap_sock:cap_sock" (at 184.15 41.91 0)
-      (effects (font (size 1.27 1.27)) hide)
-    )
-    (property "Datasheet" "~" (at 184.15 41.91 0)
+  (symbol (lib_id "Connector:TestPoint") (at 27.94 110.49 0) (unit 1)
+    (in_bom yes) (on_board yes) (dnp no) (fields_autoplaced)
+    (property "Reference" "TP1" (at 30.48 105.918 0)
+      (effects (font (size 1.27 1.27)) (justify left))
+    )
+    (property "Value" "TOUCH1" (at 30.48 108.458 0)
+      (effects (font (size 1.27 1.27)) (justify left))
+    )
+    (property "Footprint" "cap_sock:cap_sock" (at 33.02 110.49 0)
+      (effects (font (size 1.27 1.27)) hide)
+    )
+    (property "Datasheet" "~" (at 33.02 110.49 0)
       (effects (font (size 1.27 1.27)) hide)
     )
@@
     )
   )
-  (symbol (lib_id "Connector:TestPoint") (at 224.79 41.91 0) (unit 1)
-    (in_bom yes) (on_board yes) (dnp no) (fields_autoplaced)
-    (property "Reference" "TP3" (at 227.33 37.338 0)
-      (effects (font (size 1.27 1.27)) (justify left))
-    )
-    (property "Value" "TOUCH3" (at 227.33 39.878 0)
-      (effects (font (size 1.27 1.27)) (justify left))
-    )
-    (property "Footprint" "cap_sock:cap_sock" (at 229.87 41.91 0)
-      (effects (font (size 1.27 1.27)) hide)
-    )
-    (property "Datasheet" "~" (at 229.87 41.91 0)
-      (effects (font (size 1.27 1.27)) hide)
-    )
+  (symbol (lib_id "Connector:TestPoint") (at 73.66 110.49 0) (unit 1)
+    (in_bom yes) (on_board yes) (dnp no) (fields_autoplaced)
+    (property "Reference" "TP3" (at 76.2 105.918 0)
+      (effects (font (size 1.27 1.27)) (justify left))
+    )
+    (property "Value" "TOUCH3" (at 76.2 108.458 0)
+      (effects (font (size 1.27 1.27)) (justify left))
+    )
+    (property "Footprint" "cap_sock:cap_sock" (at 78.74 110.49 0)
+      (effects (font (size 1.27 1.27)) hide)
+    )
+    (property "Datasheet" "~" (at 78.74 110.49 0)
+      (effects (font (size 1.27 1.27)) hide)
+    )
